Commit message: my_robot1_description urdf

File: src/my_robot1_description/urdf/iRobot.urdf (robot description, URDF)
Before this commit: robot iRobot, 11 links, 10 joints
Links:
- removed link hokuyo_laser_link
- added link base_scan, mass 1e-5; collision cylinder length=0.04 radius=0.045; visual cylinder length=0.04 radius=0.045
Joints:
- joint hokuyo_laser_joint: child hokuyo_laser_link -> base_scan
