Commit message: my_robot1.urdf removed unused links

File: src/my_robot1_description/urdf/my_robot1.urdf (robot description, URDF)
Before this commit: robot my_robot, 7 links, 6 joints
Links:
- removed link base_footprint
- removed link caster_wheel_back_link
- removed link caster_wheel_front_link
- removed link left_wheel_link
- removed link right_wheel_link
Joints:
- removed joint base_caster_wheel_back_joint
- removed joint base_caster_wheel_front_joint
- removed joint base_joint
- removed joint base_left_wheel_joint
- removed joint base_right_wheel_joint

Commit message: nav working

File: src/my_robot1_description/urdf/my_robot1.urdf (robot description, URDF)
Before this commit: robot my_robot, 2 links, 1 joints
Links:
- added link base_footprint
Joints:
- added joint base_joint: type fixed, parent base_footprint, child base_link, origin xyz=0 0 0.036 rpy=0 0 0
- joint base_scan_joint: origin xyz=0 0 0.08 rpy=0 0 0 -> xyz=0 0 0.07 rpy=0 0 0
